File: 445L Lab 6/main.sch (EAGLE design)
At the start: 45 parts, among them IC1 LM2937, IC2 LM4041CILPRLP, Q1 16MHz, U1 TM4C1233H6PM, U2 TPA731D, U3 TLV5616

Commit message: Finished layout
Parts:
- removed Q1: 16MHz, adafruit:CRYSTALHC49U-V
- added X1: 16MHz, adafruit:XTALNX8045
- C10, C11, C14, C5, C7: device rcl:C-US050-075X075 -> resistor:CPOL-USD
- renumbered TP_GND1 to G1, TP_GND2 to G2, TP_VCC to VCC, TP_VIN to VIN
Connections:
- net 5V_IN: now also C11.+; no longer C11.1
- net GND: now also C10.-, C11.-, C14.-, C5.-, C7.-; no longer C10.2, C11.2, C14.2, C5.2, C7.2
- net OSC0: now also X1.P$2; no longer Q1.1
- net OSC1: now also X1.P$1; no longer Q1.2
- net VCC: now also C10.+, C14.+; no longer C10.1, C14.1
- net VDDC: now also C5.+, C7.+; no longer C5.1, C7.1
Other:
- moved on the sheet: C13

Commit message: Added lbr for dip-8
Parts:
- added U$1: DIP-8, lab_6:DIP-8
Changed lines of the file:
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@@
 <part name="BTN4" library="jumper" library_urn="urn:adsk.eagle:library:252" deviceset="JP1Q" device="" package3d_urn="urn:adsk.eagle:package:15455/1"/>
 <part name="X1" library="adafruit" deviceset="XTAL" device="NX8045" value="16MHz"/>
+<part name="U$1" library="lab_6" deviceset="DIP-8" device=""/>
 </parts>
 <sheets>
