File: Arduino Nano++ Square/main.brd (EAGLE design)
At the start: 83.8 x 47 mm, 68 parts, among them IC1 LM358N, Q1 IRF9530, Q2 IRF9530

Commit message: Misc updates to lab 6
Parts:
- moved R6 8.98 mm to (71.1, 21.6), turned to 0 degrees
Routing:
- net 3V3': track 60.6 -> 39.8 mm
Changed lines of the file:
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@@
 <element name="R4" library="rcl" library_urn="urn:adsk.eagle:library:334" package="0204/7" package3d_urn="urn:adsk.eagle:package:23498/1" value="10k" x="99.06" y="30.48" rot="R90"/>
 <element name="R5" library="rcl" library_urn="urn:adsk.eagle:library:334" package="0204/7" package3d_urn="urn:adsk.eagle:package:23498/1" value="10k" x="82.55" y="26.67" rot="R180"/>
-<element name="R6" library="rcl" library_urn="urn:adsk.eagle:library:334" package="0204/7" package3d_urn="urn:adsk.eagle:package:23498/1" value="" x="64.77" y="15.24" rot="R270"/>
+<element name="R6" library="rcl" library_urn="urn:adsk.eagle:library:334" package="0204/7" package3d_urn="urn:adsk.eagle:package:23498/1" value="" x="71.12" y="21.59"/>
 <element name="R7" library="rcl" library_urn="urn:adsk.eagle:library:334" package="0204/7" package3d_urn="urn:adsk.eagle:package:23498/1" value="" x="67.31" y="15.24" rot="R90"/>
 <element name="R8" library="rcl" library_urn="urn:adsk.eagle:library:334" package="0204/7" package3d_urn="urn:adsk.eagle:package:23498/1" value="300" x="95.25" y="24.13" rot="R180"/>
@@
 <wire x1="90.17" y1="39.37" x2="87.63" y2="36.83" width="1.27" layer="1"/>
 <wire x1="87.63" y1="36.83" x2="86.36" y2="36.83" width="1.27" layer="1"/>
-<wire x1="86.36" y1="36.83" x2="87.63" y2="36.83" width="0.3048" layer="16"/>
-<wire x1="87.63" y1="36.83" x2="88.9" y2="35.56" width="0.3048" layer="16"/>
-<wire x1="88.9" y1="24.765" x2="88.9" y2="35.56" width="0.3048" layer="16"/>
-<wire x1="64.77" y1="11.43" x2="63.5" y2="12.7" width="0.3048" layer="16"/>
-<wire x1="63.5" y1="12.7" x2="63.5" y2="19.685" width="0.3048" layer="16"/>
-<wire x1="63.5" y1="19.685" x2="64.135" y2="20.32" width="0.3048" layer="16"/>
-<wire x1="64.135" y1="20.32" x2="84.455" y2="20.32" width="0.3048" layer="16"/>
-<wire x1="84.455" y1="20.32" x2="88.9" y2="24.765" width="0.3048" layer="16"/>
+<wire x1="74.93" y1="21.59" x2="85.725" y2="21.59" width="0.3048" layer="16"/>
+<wire x1="85.725" y1="21.59" x2="89.535" y2="25.4" width="0.3048" layer="16"/>
+<wire x1="89.535" y1="25.4" x2="89.535" y2="34.29" width="0.3048" layer="16"/>
+<wire x1="89.535" y1="34.29" x2="86.995" y2="36.83" width="0.3048" layer="16"/>
+<wire x1="86.995" y1="36.83" x2="86.36" y2="36.83" width="0.3048" layer="16"/>
 </signal>
 <signal name="3V3EN">
@@
 <contactref element="R7" pad="2"/>
 <wire x1="69.85" y1="19.05" x2="67.31" y2="19.05" width="0.3048" layer="16"/>
-<wire x1="67.31" y1="19.05" x2="64.77" y2="19.05" width="0.3048" layer="16"/>
+<wire x1="67.31" y1="19.05" x2="67.31" y2="21.59" width="0.3048" layer="16"/>
 </signal>
 <signal name="N$2">
